Commit message: hull for multirotors

File: rotors_description/urdf/component_snippets.xacro (robot description, xacro)
@@ -681,5 +681,5 @@
       </visual>
       <inertial>
-        <mass value="0.13" />
+        <mass value="0.000013" />
         <origin xyz="0 0 0" rpy="0 0 0" />
         <inertia ixx="1e-6" ixy="0" ixz="0" iyy="1e-6" iyz="0" izz="1e-6" />
